File: esp_snapclient_v2/esp_snapclient_v2.kicad_pcb (KiCad board)
At the start: 2 copper layers, 30 parts, among them J1 USB_C_Receptacle_PowerOnly_6P, J2 Screw_Terminal_01x04, J3 Conn_01x04_Socket, SW1 SW_Push, SW2 SW_Push, U1 ESP32-WROVER-E, U2 MAX98357A, U3 MAX98357A, U5 AMS1117-3.3

Commit message: feat: up
Parts:
- removed C1: 22uF, Capacitor_SMD:C_0805_2012Metric
- removed C4: 0.1uF, Capacitor_SMD:C_0805_2012Metric
- removed R2: 0R, Resistor_SMD:R_0805_2012Metric
- moved D1 59.0 mm to (103.5, 49.0), turned to 180 degrees
- moved R5 40.6 mm to (107.5, 51.5), turned to 180 degrees
- moved R3 40.6 mm to (107.4, 49.0)
- moved C6 34.9 mm to (103.5, 51.5)
- moved C9 33.3 mm to (148.6, 51.0)
- moved C10 33.3 mm to (148.6, 54.0)
- moved C7 33.3 mm to (148.6, 45.0)
- moved C8 33.3 mm to (148.6, 48.0)
- moved R1 30.3 mm to (107.5, 63.5), turned to 180 degrees
- moved C5 29.9 mm to (103.5, 66.0)
- moved R6 28.9 mm to (161.0, 55.9), turned to 90 degrees
- moved C2 26.7 mm to (103.5, 63.5)
- moved C3 23.4 mm to (107.5, 66.0)
- moved R7 19.2 mm to (161.0, 59.6), turned to 90 degrees
- moved SW1 14.9 mm to (117.0, 80.5)
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Connections:
- SW1 pad 1: GND -> /EN
- SW1 pad 2: Net-(C4-Pad2) -> GND

Commit message: feat: up
Parts:
- added C1: 22uF, Capacitor_SMD:C_0805_2012Metric, F.Cu at (94.8, 69.6)
- moved Boot 56.6 mm to (104.9, 44.9)
- moved R6 52.3 mm to (110.5, 69.6), turned to 180 degrees
- moved J2 47.9 mm to (120.2, 43.7), turned to -90 degrees
- moved D2 47.5 mm to (113.6, 67.2), turned to 0 degrees
- moved R7 47.2 mm to (114.9, 69.6), turned to 180 degrees
- moved J1 46.4 mm to (122.2, 67.7)
- moved R8 45.7 mm to (106.2, 51.0), turned to 90 degrees
- moved R4 43.0 mm to (105.0, 48.0)
- moved U2 42.8 mm to (112.3, 43.2)
- moved R9 41.3 mm to (106.5, 64.0), turned to 90 degrees
- moved C9 37.4 mm to (112.3, 60.3), turned to 180 degrees
- moved C10 36.5 mm to (112.3, 58.2), turned to 180 degrees
- moved C7 36.2 mm to (112.4, 46.5), turned to 180 degrees
- moved C8 36.2 mm to (112.4, 49.3), turned to 180 degrees
- moved U3 33.0 mm to (112.4, 54.3)
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- renumbered SW2 to Boot
Connections:
- U2 pad 10: Net-(J2-Pin_2) -> Net-(J2-Pin_1)
- U2 pad 9: Net-(J2-Pin_1) -> Net-(J2-Pin_2)
- U3 pad 10: Net-(J2-Pin_4) -> Net-(J2-Pin_3)
- U3 pad 9: Net-(J2-Pin_3) -> Net-(J2-Pin_4)
Routing:
- net +3V3: track 0.00 -> 81.9 mm, vias 0 -> 4
- net GND: track 0.00 -> 81.6 mm, vias 0 -> 8
- net +5V: track 0.00 -> 66.7 mm, vias 0 -> 2
- net /GPIO25: track 0.00 -> 53.4 mm, vias 0 -> 3
- net /GPIO26: track 0.00 -> 48.6 mm, vias 0 -> 3
- net /GPIO27: track 0.00 -> 44.9 mm, vias 0 -> 3
- net /GPIO18: track 0.00 -> 27.5 mm
- net /EN: track 0.00 -> 26.1 mm
- net Net-(U3-GAIN_SLOT): track 0.00 -> 13.9 mm, vias 0 -> 2
- net /RX: track 0.00 -> 12.8 mm
- net /TX: track 0.00 -> 11.6 mm
- net Net-(U3-~{SD_MODE}): track 0.00 -> 11.2 mm, vias 0 -> 2
- net Net-(U1-GPIO0/BOOT/ADC2_CH1): track 0.00 -> 11.1 mm
- net Net-(U2-GAIN_SLOT): track 0.00 -> 10.6 mm, vias 0 -> 2
- net Net-(J1-CC2): track 0.00 -> 8.70 mm
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- added copper zone on B.Cu, net GND
- added copper zone on F.Cu, net GND
Other:
- board outline added: 49 x 33.3 mm
- board text added: "3V3"
- board text added: "Boot"
- board text added: "EN"
- board text added: "GND"
- board text added: "N"
- board text added: "P"
- board text added: "RX"
- board text added: "TX"

Commit message: feat: up
Parts:
- J3: value Conn_01x04_Socket -> UART; footprint my-footprints:下载孔 -> Connector_PinHeader_2.54mm:PinHeader_1x04_P2.54mm_Vertical
- SW1: value SW_Push -> EN
- SW2: renamed from Boot; value SW_Push -> Boot
- turned J3 to 90 degrees
Connections:
- net Net-(U1-GPIO0/BOOT/ADC2_CH1) renamed /Boot
Routing:
- net GND: track 81.6 -> 74.7 mm, vias 8 -> 11
- net /EN: track 26.1 -> 31.0 mm, vias 0 -> 3
- net +3V3: track 81.9 -> 78.1 mm
Other:
- board size 49 x 33.3 mm -> 49 x 35 mm

Commit message: feat: up
Parts:
- J2: value Screw_Terminal_01x04 -> Speaker
- moved C6 2.90 mm to (106.8, 51.0)
- moved R8 2.40 mm to (103.8, 51.0)
Connections:
- R8 pad 1: +5V -> GND
- R9 pad 1: +5V -> GND
Routing:
- net +5V: track 66.7 -> 56.3 mm, vias 2 -> 0
- net GND: track 74.7 -> 78.9 mm
- net Net-(U2-GAIN_SLOT): track 10.6 -> 13.7 mm
Changed lines of the file:
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@@
 			)
 		)
-		(property "Value" "Screw_Terminal_01x04"
+		(property "Value" "Speaker"
 			(at 8.51 5.0675 90)
 			(layer "F.Fab")
@@
 	(footprint "Capacitor_SMD:C_0805_2012Metric"
 		(layer "F.Cu")
-		(at 103.9 51 90)
+		(at 106.8 50.95 90)
 		(descr "Capacitor SMD 0805 (2012 Metric), square (rectangular) end terminal, IPC-7351 nominal, (Body size source: IPC-SM-782 page 76, https://www.pcb-3d.com/wordpress/wp-content/uploads/ipc-sm-782a_amendment_1_and_2.pdf, https://docs.google.com/spreadsheets/d/1BsfQQcO9C6DZCsRaXUlFlo91Tg2WpOkGARC1WS5S8t0/edit?usp=sharing), generated with kicad-footprint-generator")
 		(tags "capacitor")
@@
 			(at 0 1.68 90)
 			(layer "F.Fab")
+			(hide yes)
 			(effects
 				(font
@@
 	(footprint "Resistor_SMD:R_0805_2012Metric"
 		(layer "F.Cu")
-		(at 106.2 51 90)
+		(at 103.8 51.0125 90)
 		(descr "Resistor SMD 0805 (2012 Metric), square (rectangular) end terminal, IPC-7351 nominal, (Body size source: IPC-SM-782 page 72, https://www.pcb-3d.com/wordpress/wp-content/uploads/ipc-sm-782a_amendment_1_and_2.pdf), generated with kicad-footprint-generator")
 		(tags "resistor")
@@
 			(layers "F.Cu" "F.Mask" "F.Paste")
 			(roundrect_rratio 0.243902)
-			(net 4 "+5V")
+			(net 2 "GND")
 			(pintype "passive")
 		)
@@
 			(layers "F.Cu" "F.Mask" "F.Paste")
 			(roundrect_rratio 0.243902)
-			(net 4 "+5V")
+			(net 2 "GND")
 			(pintype "passive")
 		)
@@
 	)
 	(segment
-		(start 103.25 50.05)
-		(end 102.2 51.1)
+		(start 106.8 50)
+		(end 104.875 51.925)
+		(width 0.25)
+		(layer "F.Cu")
+		(net 2)
+	)
+	(segment
+		(start 103.8 51.925)
+		(end 103.025 51.925)
 		(width 0.25)
 		(layer "F.Cu")
@@
 	)
 	(segment
+		(start 106.5 64.9125)
+		(end 107.0875 64.9125)
+		(width 0.25)
+		(layer "F.Cu")
+		(net 2)
+	)
+	(segment
 		(start 112.1 41.725)
 		(end 112.1 41.261346)
@@
 	)
 	(segment
+		(start 103.025 51.925)
+		(end 102.2 51.1)
+		(width 0.25)
+		(layer "F.Cu")
+		(net 2)
+	)
+	(segment
 		(start 107.9 45.7)
 		(end 107.1 44.9)
@@
 	)
 	(segment
-		(start 113.8275 54.06)
-		(end 114.679702 54.06)
+		(start 104.875 51.925)
+		(end 103.8 51.925)
 		(width 0.25)
 		(layer "F.Cu")
@@
 	)
 	(segment
-		(start 103.9 50.05)
-		(end 103.25 50.05)
+		(start 113.8275 54.06)
+		(end 114.679702 54.06)
 		(width 0.25)
 		(layer "F.Cu")
@@
 	)
 	(segment
-		(start 107.0875 64.9125)
-		(end 107.9 64.1)
-		(width 0.25)
+		(start 106.8 51.9)
+		(end 105.801 52.899)
+		(width 0.5)
 		(layer "F.Cu")
 		(net 4)
@@
 	)
 	(segment
-		(start 103.9 53.25)
+		(start 105.801 52.899)
+		(end 104.251 52.899)
+		(width 0.5)
+		(layer "F.Cu")
+		(net 4)
+	)
+	(segment
+		(start 104.251 52.899)
 		(end 102.8 54.35)
 		(width 0.5)
@@
 	)
 	(segment
-		(start 106.5875 51.9125)
-		(end 107.9 50.6)
-		(width 0.5)
-		(layer "F.Cu")
-		(net 4)
-	)
-	(segment
 		(start 115.5575 66.18)
 		(end 114.5375 67.2)
@@
 	)
 	(segment
-		(start 103.9 51.95)
-		(end 103.9 53.25)
-		(width 0.5)
-		(layer "F.Cu")
-		(net 4)
-	)
-	(segment
 		(start 119.766924 69.22)
 		(end 120.296 68.690924)
@@
 	)
 	(segment
-		(start 107.9 50.6)
-		(end 113.6 50.6)
-		(width 0.5)
-		(layer "F.Cu")
-		(net 4)
-	)
-	(segment
 		(start 119.12 69.22)
 		(end 119.766924 69.22)
@@
 	)
 	(segment
-		(start 120.296 68.690924)
-		(end 120.296 66.709076)
-		(width 0.75)
+		(start 106.8 51.9)
+		(end 107.95375 50.74625)
+		(width 0.5)
 		(layer "F.Cu")
 		(net 4)
 	)
 	(segment
-		(start 103.9 51.95)
-		(end 106.1625 51.95)
-		(width 0.5)
+		(start 120.296 68.690924)
+		(end 120.296 66.709076)
+		(width 0.75)
 		(layer "F.Cu")
 		(net 4)
@@
 	)
 	(segment
-		(start 106.5 64.9125)
-		(end 107.0875 64.9125)
-		(width 0.25)
-		(layer "F.Cu")
-		(net 4)
-	)
-	(segment
 		(start 114.85375 50.74625)
 		(end 114.15375 50.04625)
@@
 	)
 	(segment
-		(start 115.7 64.6)
-		(end 114.9125 64.6)
-		(width 0.25)
-		(layer "F.Cu")
-		(net 4)
-	)
-	(segment
 		(start 119.12 66.18)
 		(end 115.5575 66.18)
@@
 	)
 	(segment
-		(start 114.5125 65)
-		(end 114.5125 62.8)
-		(width 0.75)
-		(layer "F.Cu")
-		(net 4)
-	)
-	(segment
-		(start 113.6 50.6)
-		(end 114.15375 50.04625)
+		(start 107.95375 50.74625)
+		(end 114.85375 50.74625)
 		(width 0.5)
 		(layer "F.Cu")
 		(net 4)
 	)
-	(via
-		(at 115.7 64.6)
-		(size 0.6)
-		(drill 0.3)
-		(layers "F.Cu" "B.Cu")
-		(net 4)
-	)
-	(via
-		(at 107.9 64.1)
-		(size 0.6)
-		(drill 0.3)
-		(layers "F.Cu" "B.Cu")
-		(net 4)
-	)
-	(segment
-		(start 115.2 64.1)
-		(end 115.7 64.6)
-		(width 0.25)
-		(layer "B.Cu")
-		(net 4)
-	)
 	(segment
-		(start 107.9 64.1)
-		(end 115.2 64.1)
-		(width 0.25)
-		(layer "B.Cu")
+		(start 114.5125 65)
+		(end 114.5125 62.8)
+		(width 0.75)
+		(layer "F.Cu")
 		(net 4)
 	)
@@
 	)
 	(segment
-		(start 108.1 49.4)
-		(end 106.8875 49.4)
+		(start 110.9125 42.9125)
+		(end 109.6125 42.9125)
 		(width 0.25)
 		(layer "F.Cu")
@@
 	)
 	(segment
-		(start 106.8875 49.4)
-		(end 106.2 50.0875)
+		(start 104.726 49.174)
+		(end 108.326 49.174)
 		(width 0.25)
 		(layer "F.Cu")
@@
 	)
 	(segment
-		(start 110.9125 42.9125)
-		(end 109.6125 42.9125)
+		(start 103.8 50.1)
+		(end 104.726 49.174)
 		(width 0.25)
 		(layer "F.Cu")
@@
 	)
 	(segment
-		(start 109.6 47.9)
-		(end 108.1 49.4)
+		(start 103.9 50.05)
+		(end 103.25 50.05)
 		(width 0.25)
 		(layer "F.Cu")
@@
 		(width 0.25)
 		(layer "F.Cu")
+		(net 17)
+	)
+	(segment
+		(start 108.326 49.174)
+		(end 109.6 47.9)
+		(width 0.25)
+		(layer "F.Cu")
