File: esp_snapclient_v2/esp_snapclient_v2.kicad_sch (KiCad schematic)
At the start: 13 parts, among them SW1 SW_Push, SW2 SW_Push, U1 ESP32-WROVER-E, U2 MAX98357A, U3 MAX98357A

Commit message: feat: up
Parts:
- added C5, C6: 22uF, Capacitor_SMD:C_0805_2012Metric, symbol Device:C
- added D1: LED, symbol Device:LED
- added J1: USB_C_Receptacle_PowerOnly_6P, symbol Connector:USB_C_Receptacle_PowerOnly_6P
- added R5: 2K, Resistor_SMD:R_0805_2012Metric, symbol Device:R
- added R6, R7: 5.1K, Resistor_SMD:R_0805_2012Metric, symbol Device:R
- added U5: AMS1117-3.3, Package_TO_SOT_SMD:SOT-223-3_TabPin2, symbol Regulator_Linear:AMS1117-3.3
Connections:
- net +3V3: now also C5.1, U5.2 (VO)
- net GND: now also C5.2, C6.2, D1.1 (K), J1.A12 (GND), J1.B12 (GND), J1.S1 (SHIELD), R6.2, R7.2, U5.1 (GND)
- new net: J1.A5 (CC1), R7.1
- new net: D1.2 (A), R5.2
- new net: J1.B5 (CC2), R6.1
- new net +5V: C6.1, J1.A9 (VBUS), J1.B9 (VBUS), R5.1, U5.3 (VI)
Other:
- moved on the sheet: C1, C2, C3, C4, R1, R2, R3, R4, SW1, SW2, U1, U2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

Commit message: feat: up
Parts:
- added C10, C7: 0.1uF, Capacitor_SMD:C_0805_2012Metric, symbol Device:C
- added C8, C9: 10uF, Capacitor_SMD:C_0805_2012Metric, symbol Device:C
- added D2: ESD9B3.3ST5G, Diode_SMD:D_0805_2012Metric, symbol Diode:ESD9B3.3ST5G
- added J2: Screw_Terminal_01x04, TerminalBlock:TerminalBlock_MaiXu_MX126-5.0-04P_1x04_P5.00mm, symbol Connector:Screw_Terminal_01x04
- added J3: Conn_01x04_Socket, my-footprints:下载孔, symbol Connector:Conn_01x04_Socket
- added R8, R9: 100K, Resistor_SMD:R_0805_2012Metric, symbol Device:R
- D1: footprint (none) -> LED_SMD:LED_0805_2012Metric
- J1: footprint (none) -> Connector_USB:USB_C_Receptacle_GCT_USB4125-xx-x-0190_6P_TopMnt_Horizontal
Connections:
- net +3V3: now also J3.1 (Pin_1)
- net +5V: now also U2.7 (VDD), U2.8 (VDD), U3.7 (VDD), U3.8 (VDD), C10.1, C7.1, C8.1, C9.1, D2.2 (A2), R8.1, R9.1
- net GND: now also U2.11 (GND), U2.15 (GND), U2.3 (GND), U3.11 (GND), U3.15 (GND), U3.3 (GND), C10.2, C7.2, C8.2, C9.2, D2.1 (A1), J3.4 (Pin_4)
- net GPIO27: now reaches U2.1 (DIN), U3.1 (DIN)
- net GPIO27: now also U1.12 (ADC2_CH7/GPIO27)
- net at U2.10 (OUTN): now also J2.2 (Pin_2)
- net GPIO25: now reaches U2.14 (LRCLK), U3.14 (LRCLK)
- net GPIO25: now also U1.10 (DAC_1/ADC2_CH8/GPIO25)
- net GPIO26: now reaches U2.16 (BCLK), U3.16 (BCLK)
- net GPIO26: now also U1.11 (DAC_2/ADC2_CH9/GPIO26)
- net at U2.2 (GAIN_SLOT): now also R8.2
- net at U2.9 (OUTP): now also J2.1 (Pin_1)
- net RX: now reaches U1.34 (U0RXD/GPIO3)
- net RX: now also J3.3 (Pin_3)
- net TX: now reaches U1.35 (U0TXD/GPIO1)
- net TX: now also J3.2 (Pin_2)
- net at U3.10 (OUTN): now also J2.4 (Pin_4)
- net at U3.2 (GAIN_SLOT): now also R9.2
- net at U3.9 (OUTP): now also J2.3 (Pin_3)
- no-connect marks 0 -> 19
Other:
- moved on the sheet: J1, R3, R4, R6, R7, SW2, U1, U3

Commit message: feat: up
Parts:
- removed C1: 22uF, Capacitor_SMD:C_0805_2012Metric, symbol Device:C
- removed C4: 0.1uF, Capacitor_SMD:C_0805_2012Metric, symbol Device:C
- removed R2: 0R, Resistor_SMD:R_0805_2012Metric, symbol Device:R
Connections:
- net EN: now also SW1.1
- net GND: now also SW1.2; no longer SW1.1
Other:
- moved on the sheet: SW1

Commit message: feat: up
Parts:
- added C1: 22uF, Capacitor_SMD:C_0805_2012Metric, symbol Device:C
Connections:
- net +3V3: now also C1.1
- net GND: now also C1.2
- net at U2.10 (OUTN): now also J2.1 (Pin_1); no longer J2.2 (Pin_2)
- net at U2.9 (OUTP): now also J2.2 (Pin_2); no longer J2.1 (Pin_1)
- net at U3.10 (OUTN): now also J2.3 (Pin_3); no longer J2.4 (Pin_4)
- net at U3.9 (OUTP): now also J2.4 (Pin_4); no longer J2.3 (Pin_3)

Commit message: feat: up
Parts:
- J2: value Screw_Terminal_01x04 -> Speaker
- J3: value Conn_01x04_Socket -> UART; footprint my-footprints:下载孔 -> Connector_PinHeader_2.54mm:PinHeader_1x04_P2.54mm_Vertical
- SW1: value SW_Push -> EN
- SW2: value SW_Push -> Boot
Connections:
- net Boot: now reaches R3.1, SW2.1, U1.25 (GPIO0/BOOT/ADC2_CH1)
Other:
- moved on the sheet: C1, C2, C3, C5, C6, D1, J3, R1, R3, R5, SW1, SW2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

Commit message: feat: up
Connections:
- net +5V: no longer R8.1, R9.1
- net GND: now also R8.1, R9.1
Changed lines of the file:
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@@
+	)
+	(symbol
+		(lib_id "power:GND")
+		(at 224.79 156.21 0)
+		(unit 1)
+		(exclude_from_sim no)
+		(in_bom yes)
+		(on_board yes)
+		(dnp no)
+		(fields_autoplaced yes)
+		(property "Reference" "#PWR05"
+			(at 224.79 162.56 0)
+			(effects
+				(font
+					(size 1.27 1.27)
+				)
+				(hide yes)
+			)
+		)
+		(property "Value" "GND"
+			(at 224.79 161.29 0)
+			(effects
+				(font
+					(size 1.27 1.27)
+				)
+			)
+		)
+		(property "Footprint" ""
+			(at 224.79 156.21 0)
+			(effects
+				(font
+					(size 1.27 1.27)
+				)
+				(hide yes)
+			)
+		)
+		(property "Datasheet" ""
+			(at 224.79 156.21 0)
+			(effects
+				(font
+					(size 1.27 1.27)
+				)
+				(hide yes)
+			)
+		)
+		(property "Description" "Power symbol creates a global label with name \"GND\" , ground"
+			(at 224.79 156.21 0)
+			(effects
+				(font
+					(size 1.27 1.27)
+				)
+				(hide yes)
+			)
+		)
+		(pin "1"
+		)
+		(instances
+			(project ""
+				(path "/6793efc9-4502-4797-8f8c-dbe7d1c802c7"
+					(reference "#PWR05")
+					(unit 1)
+				)
+			)
+		)
 	)
 	(symbol
@@
 	)
 	(symbol
-		(lib_id "power:+5V")
-		(at 199.39 105.41 90)
-		(unit 1)
-		(exclude_from_sim no)
-		(in_bom yes)
-		(on_board yes)
-		(dnp no)
-		(fields_autoplaced yes)
-		(property "Reference" "#PWR019"
-			(at 203.2 105.41 0)
-			(effects
-				(font
-					(size 1.27 1.27)
-				)
-				(hide yes)
-			)
-		)
-		(property "Value" "+5V"
-			(at 195.58 105.4099 90)
-			(effects
-				(font
-					(size 1.27 1.27)
-				)
-				(justify left)
-			)
-		)
-		(property "Footprint" ""
-			(at 199.39 105.41 0)
-			(effects
-				(font
-					(size 1.27 1.27)
-				)
-				(hide yes)
-			)
-		)
-		(property "Datasheet" ""
-			(at 199.39 105.41 0)
-			(effects
-				(font
-					(size 1.27 1.27)
-				)
-				(hide yes)
-			)
-		)
-		(property "Description" "Power symbol creates a global label with name \"+5V\""
-			(at 199.39 105.41 0)
-			(effects
-				(font
-					(size 1.27 1.27)
-				)
-				(hide yes)
-			)
-		)
-		(pin "1"
-		)
-		(instances
-			(project ""
-				(path "/6793efc9-4502-4797-8f8c-dbe7d1c802c7"
-					(reference "#PWR019")
-					(unit 1)
-				)
-			)
-		)
-	)
-	(symbol
 		(lib_id "power:GND")
 		(at 231.14 130.81 0)
@@
 	)
 	(symbol
-		(lib_id "power:+5V")
-		(at 224.79 156.21 90)
-		(unit 1)
-		(exclude_from_sim no)
-		(in_bom yes)
-		(on_board yes)
-		(dnp no)
-		(fields_autoplaced yes)
-		(property "Reference" "#PWR020"
-			(at 228.6 156.21 0)
-			(effects
-				(font
-					(size 1.27 1.27)
-				)
-				(hide yes)
-			)
-		)
-		(property "Value" "+5V"
-			(at 220.98 156.2099 90)
-			(effects
-				(font
-					(size 1.27 1.27)
-				)
-				(justify left)
-			)
-		)
-		(property "Footprint" ""
-			(at 224.79 156.21 0)
-			(effects
-				(font
-					(size 1.27 1.27)
-				)
-				(hide yes)
-			)
-		)
-		(property "Datasheet" ""
-			(at 224.79 156.21 0)
-			(effects
-				(font
-					(size 1.27 1.27)
-				)
-				(hide yes)
-			)
-		)
-		(property "Description" "Power symbol creates a global label with name \"+5V\""
-			(at 224.79 156.21 0)
-			(effects
-				(font
-					(size 1.27 1.27)
-				)
-				(hide yes)
-			)
-		)
-		(pin "1"
-		)
-		(instances
-			(project ""
-				(path "/6793efc9-4502-4797-8f8c-dbe7d1c802c7"
-					(reference "#PWR020")
-					(unit 1)
-				)
-			)
-		)
-	)
-	(symbol
 		(lib_id "Connector:USB_C_Receptacle_PowerOnly_6P")
 		(at 34.29 33.02 0)
@@
 					(unit 1)
 				)
+			)
+		)
+	)
+	(symbol
+		(lib_id "power:GND")
+		(at 199.39 105.41 0)
+		(unit 1)
+		(exclude_from_sim no)
+		(in_bom yes)
+		(on_board yes)
+		(dnp no)
+		(fields_autoplaced yes)
+		(property "Reference" "#PWR03"
+			(at 199.39 111.76 0)
+			(effects
+				(font
+					(size 1.27 1.27)
+				)
+				(hide yes)
+			)
+		)
+		(property "Value" "GND"
+			(at 199.39 110.49 0)
+			(effects
+				(font
+					(size 1.27 1.27)
+				)
+			)
+		)
+		(property "Footprint" ""
+			(at 199.39 105.41 0)
+			(effects
+				(font
+					(size 1.27 1.27)
+				)
+				(hide yes)
+			)
+		)
+		(property "Datasheet" ""
+			(at 199.39 105.41 0)
+			(effects
+				(font
+					(size 1.27 1.27)
+				)
+				(hide yes)
+			)
+		)
+		(property "Description" "Power symbol creates a global label with name \"GND\" , ground"
+			(at 199.39 105.41 0)
+			(effects
+				(font
+					(size 1.27 1.27)
+				)
+				(hide yes)
+			)
+		)
+		(pin "1"
+		)
+		(instances
+			(project ""
+				(path "/6793efc9-4502-4797-8f8c-dbe7d1c802c7"
+					(reference "#PWR03")
+					(unit 1)
+				)
