File: wled/wled.kicad_pcb (KiCad board)
At the start: 2 copper layers, 31 parts, among them J1 UART, J2 USB_C_Receptacle_PowerOnly_6P, J3 LED PIN, SW1 EN, SW2 Boot, U1 ESP32-C3-MINI-1, U2 AMS1117-3.3

Commit message: feat: up
Parts:
- removed R3: 0, Resistor_SMD:R_0805_2012Metric
- moved J1 128.8 mm to (101.0, 52.0), turned to 90 degrees
- moved MK2 126.7 mm to (121.5, 69.0), turned to 90 degrees
- moved R10 126.1 mm to (112.9, 66.4), turned to 180 degrees
- moved R9 126.1 mm to (113.0, 63.9), turned to 180 degrees
- moved SW1 122.1 mm to (127.3, 52.0)
- moved MK1 122.1 mm to (121.5, 52.0), turned to 90 degrees
- moved D2 121.8 mm to (126.4, 58.1)
- moved D1 121.6 mm to (126.4, 61.1)
- moved SW2 119.1 mm to (130.3, 57.0), turned to -90 degrees
- moved R6 114.4 mm to (126.4, 69.7), turned to 180 degrees
- moved R5 108.3 mm to (126.4, 66.8), turned to 180 degrees
- moved R4 108.3 mm to (126.4, 64.0)
- moved J2 105.3 mm to (133.5, 65.6), turned to 90 degrees
- moved J3 101.1 mm to (134.3, 52.4)
- moved C4 95.8 mm to (126.4, 55.2)
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Connections:
- C4 pad 2: Net-(C4-Pad2) -> /EN
- SW1 pad 2: Net-(C4-Pad2) -> /EN
Routing:
- net +3V3: track 0.00 -> 79.3 mm, vias 0 -> 3
- net +5V: track 0.00 -> 46.3 mm
- net /EN: track 0.00 -> 43.7 mm, vias 0 -> 3
- net /IO10: track 0.00 -> 36.0 mm, vias 0 -> 1
- net Net-(MK1-BCLK): track 0.00 -> 31.8 mm, vias 0 -> 3
- net GND: track 0.00 -> 27.3 mm, vias 0 -> 14
- net Net-(MK1-WS): track 0.00 -> 26.4 mm, vias 0 -> 3
- net Net-(U1-GPIO9): track 0.00 -> 25.5 mm, vias 0 -> 2
- net /IO8: track 0.00 -> 23.4 mm, vias 0 -> 3
- net Net-(U1-GPIO2/ADC1_CH2): track 0.00 -> 14.3 mm, vias 0 -> 2
- net Net-(MK2-DATA): track 0.00 -> 10.1 mm, vias 0 -> 2
- net /IO6: track 0.00 -> 8.70 mm
- net /IO7: track 0.00 -> 7.07 mm
- net Net-(J2-CC1): track 0.00 -> 5.24 mm
- net Net-(J2-CC2): track 0.00 -> 3.83 mm
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- added copper zone on B.Cu, net GND
- added copper zone on F.Cu, net GND
Other:
- board outline added: 37.4 x 22.3 mm
- board text added: "5V"
- board text added: "Boot"
- board text added: "EN"
- board text added: "GND"
- board text added: "IO10"
