File: wled/wled.kicad_sch (KiCad schematic)
At the start: 31 parts, among them J1 UART, J2 USB_C_Receptacle_PowerOnly_6P, J3 LED PIN, SW1 EN, SW2 Boot, U1 ESP32-C3-MINI-1, U2 AMS1117-3.3

Commit message: feat: up
Parts:
- removed R3: 0, Resistor_SMD:R_0805_2012Metric, symbol Device:R
Connections:
- net EN: now also C4.2, SW1.2
Changed lines of the file:
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@@
-	(wire
-		(pts
-			(xy 114.3 157.48) (xy 119.38 157.48)
-		)
-		(stroke
-			(width 0)
-			(type default)
-		)
-	)
 	(wire
 		(pts
@@
 	(wire
 		(pts
-			(xy 104.14 157.48) (xy 106.68 157.48)
+			(xy 104.14 157.48) (xy 119.38 157.48)
 		)
 		(stroke
@@
 					(unit 1)
 				)
-			)
-		)
-	)
-	(symbol
-		(lib_id "Device:R")
-		(at 110.49 157.48 90)
-		(unit 1)
-		(exclude_from_sim no)
-		(in_bom yes)
-		(on_board yes)
-		(dnp no)
-		(fields_autoplaced yes)
-		(property "Reference" "R3"
-			(at 110.49 151.13 90)
-			(effects
-				(font
-					(size 1.27 1.27)
-				)
-			)
-		)
-		(property "Value" "0"
-			(at 110.49 153.67 90)
-			(effects
-				(font
-					(size 1.27 1.27)
-				)
-			)
-		)
-		(property "Footprint" "Resistor_SMD:R_0805_2012Metric"
-			(at 110.49 159.258 90)
-			(effects
-				(font
-					(size 1.27 1.27)
-				)
-				(hide yes)
-			)
-		)
-		(property "Datasheet" "~"
-			(at 110.49 157.48 0)
-			(effects
-				(font
-					(size 1.27 1.27)
-				)
-				(hide yes)
-			)
-		)
-		(property "Description" "Resistor"
-			(at 110.49 157.48 0)
-			(effects
-				(font
-					(size 1.27 1.27)
-				)
-				(hide yes)
-			)
-		)
-		(pin "1"
-		)
-		(pin "2"
-		)
-		(instances
-			(project "wled"
-				(path "/859775a4-a02c-4bf3-9b8b-fe3e9fc7e226"
-					(reference "R3")
-					(unit 1)
-				)
